Commit message: Post URC commit

File: prochesta_arm/urdf/prochesta_arm.urdf.xacro (robot description, xacro)
@@ -40,19 +40,19 @@
         </inertial>
         <visual name="">
-            <origin xyz="0.0 0.0 0.01" rpy="0.0 0.0 0.0"/>
-            <geometry>
-                <box size="1.5 1.5 0.02"/>
+            <origin xyz="0.0 0.0 0.51" rpy="0.0 0.0 0.0"/>
+            <geometry>
+                <box size="1. 1. 0.32"/>
             </geometry>
             <material name="grey"/>
         </visual>
         <collision>
-            <origin xyz="0.0 0.0 0.01" rpy="0.0 0.0 0.0"/>
-            <geometry>
-                <box size="1.5 1.5 0.02"/>
+            <origin xyz="0.0 0.0 0.51" rpy="0.0 0.0 0.0"/>
+            <geometry>
+                <box size="1. 1. 0.32"/>
             </geometry>
         </collision>
     </link>
     <joint name="base_plane__ArmBase" type="fixed">
-        <origin rpy="0.0 0.0 0.0" xyz="0.0546412131471822 0.0 0.11" />
+        <origin rpy="0.0 0.0 0.0" xyz="0.0546412131471822 0.6 0.56" />
         <parent link="base_bar" />
         <child link="ArmBase" />
